File: attiny-devboard.kicad_pcb (KiCad board)
At the start: 2 copper layers, 48.3 x 30.5 mm, 16 parts, among them J1 POWER, J6 ICSP, U1 ATtiny85-20SU

Commit message: updates
Parts:
- removed J6: ICSP, Connector_PinHeader_2.54mm:PinHeader_2x03_P2.54mm_Vertical
- removed R3, R4, R5, R6: R, Resistor_SMD:R_0805_2012Metric_Pad1.15x1.40mm_HandSolder
- added C2: 0.1uF, Capacitor_SMD:C_0805_2012Metric_Pad1.15x1.40mm_HandSolder, F.Cu at (120.3, 83.8)
- added C3: 100u, Capacitor_SMD:C_0805_2012Metric_Pad1.15x1.40mm_HandSolder, F.Cu at (115.0, 82.9)
- added C4: .1uF, Capacitor_SMD:C_0805_2012Metric_Pad1.15x1.40mm_HandSolder, F.Cu at (139.4, 76.8)
- added D10: LED, Diode_SMD:D_0805_2012Metric_Pad1.15x1.40mm_HandSolder, F.Cu at (128.5, 96.0)
- added D11: LED, Diode_SMD:D_0805_2012Metric_Pad1.15x1.40mm_HandSolder, F.Cu at (132.7, 90.7)
- added D12: LED, Diode_SMD:D_0805_2012Metric_Pad1.15x1.40mm_HandSolder, F.Cu at (132.4, 96.0)
- added D13: LED, Diode_SMD:D_0805_2012Metric_Pad1.15x1.40mm_HandSolder, F.Cu at (136.7, 90.7)
- added D14: LED, Diode_SMD:D_0805_2012Metric_Pad1.15x1.40mm_HandSolder, F.Cu at (136.3, 96.0)
- added D15: LED, Diode_SMD:D_0805_2012Metric_Pad1.15x1.40mm_HandSolder, F.Cu at (140.6, 90.7)
- added D16: LED, Diode_SMD:D_0805_2012Metric_Pad1.15x1.40mm_HandSolder, F.Cu at (140.2, 96.0)
- added D17: LED, Diode_SMD:D_0805_2012Metric_Pad1.15x1.40mm_HandSolder, F.Cu at (107.3, 96.7)
- added D7: LED, Diode_SMD:D_0805_2012Metric_Pad1.15x1.40mm_HandSolder, F.Cu at (124.8, 90.7)
- added D8: LED, Diode_SMD:D_0805_2012Metric_Pad1.15x1.40mm_HandSolder, F.Cu at (124.6, 96.0)
- added D9: LED, Diode_SMD:D_0805_2012Metric_Pad1.15x1.40mm_HandSolder, F.Cu at (128.7, 90.7)
- added J2: ICSP, Connector_PinHeader_2.54mm:PinHeader_2x03_P2.54mm_Vertical, F.Cu at (109.7, 81.7)
- added U2: ATtiny85-20SU, Package_SO:SOIJ-8_5.3x5.3mm_P1.27mm, F.Cu at (117.7, 77.8)
- C1: value 100u -> 1uF
- D2, D3, D4, D5, D6: footprint LED_SMD:LED_0805_2012Metric -> Diode_SMD:D_0805_2012Metric_Pad1.15x1.40mm_HandSolder
- R1: value R -> 20k
- U1: value ATtiny85-20SU -> IS31FL3731-SA; footprint Package_SO:SOIJ-8_5.3x5.3mm_P1.27mm -> Package_SO:SSOP-28_5.3x10.2mm_P0.65mm
- moved D6 21.3 mm to (120.7, 96.0), turned to 50 degrees
- moved D5 19.6 mm to (120.8, 90.7), turned to 50 degrees
- moved R2 19.5 mm to (107.3, 94.1), turned to 180 degrees
- moved D4 17.9 mm to (116.8, 96.0), turned to 50 degrees
- moved D3 16.6 mm to (116.8, 90.7), turned to 50 degrees
- moved D2 14.4 mm to (112.9, 96.0), turned to 50 degrees
- moved R1 8.91 mm to (122.9, 83.8), turned to 90 degrees
- moved D1 8.34 mm to (112.9, 90.7), turned to 50 degrees
- moved J1 3.70 mm to (107.2, 86.9)
- moved C1 3.11 mm to (136.8, 76.8), turned to 90 degrees
- moved U1 0.82 mm to (129.3, 80.4), turned to 180 degrees
Connections:
- C1 pad 1: +3V3 -> GND
- C1 pad 2: GND -> +3V3
- D1 pad 1: GND -> /CA1
- D2 pad 1: GND -> /CA2
- D2 pad 2: Net-(D2-Pad2) -> Net-(D1-Pad2)
- D3 pad 1: GND -> /CA1
- D4 pad 1: GND -> /CA2
- D4 pad 2: Net-(D4-Pad2) -> Net-(D3-Pad2)
- D5 pad 1: GND -> /CA1
- D6 pad 1: GND -> /CA2
- D6 pad 2: Net-(D6-Pad2) -> Net-(D5-Pad2)
- R1 pad 1: Net-(D1-Pad2) -> GND
- R1 pad 2: +3V3 -> Net-(R1-Pad2)
- R2 pad 1: SCK -> Net-(D17-Pad2)
- R2 pad 2: Net-(D2-Pad2) -> +3V3
- U1 pad 1: RST -> Net-(U1-Pad1)
- U1 pad 2: PB3 -> +3V3
- U1 pad 3: PB4 -> Net-(U1-Pad3)
- U1 pad 4: GND -> Net-(U1-Pad4)
- U1 pad 5: MOSI -> GND
- U1 pad 6: MISO -> Net-(R1-Pad2)
- U1 pad 7: SCK -> Net-(U1-Pad7)
- U1 pad 8: +3V3 -> Net-(U1-Pad8)
Routing:
- net MISO: track 72.8 -> 6.66 mm
- net /CA1: track 0.00 -> 63.1 mm, vias 0 -> 2
- net /CA2: track 0.00 -> 60.0 mm, vias 0 -> 2
- net SCK: track 68.9 -> 26.2 mm, vias 1 -> 0
- net PB3: track 32.1 -> 0.00 mm, vias 2 -> 0
- net PB4: track 30.6 -> 0.00 mm, vias 2 -> 0
- net MOSI: track 41.0 -> 22.5 mm
- net Net-(C2-Pad1): track 0.00 -> 14.9 mm, vias 0 -> 2
- net +3V3: track 9.17 -> 22.7 mm, vias 2 -> 3
- net Net-(R1-Pad2): track 0.00 -> 13.4 mm
- net RST: track 26.9 -> 14.1 mm, vias 2 -> 0
- net Net-(D7-Pad2): track 0.00 -> 9.97 mm, vias 0 -> 2
- net Net-(D10-Pad2): track 0.00 -> 9.73 mm, vias 0 -> 2
- net Net-(D11-Pad2): track 0.00 -> 9.66 mm, vias 0 -> 2
- net Net-(D13-Pad2): track 0.00 -> 9.33 mm, vias 0 -> 2
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Other:
- board text removed: "attiny85 devboard 7/20/2020 v2.2"
