File: attiny-devboard.sch (KiCad schematic (older format))
At the start: 16 parts, among them J1 POWER, J6 ICSP, U1 ATtiny85-20SU

Commit message: updates
Parts:
- removed R2, R3, R4, R5, R6: R, Resistor_SMD:R_0805_2012Metric_Pad1.15x1.40mm_HandSolder, symbol Device:R
- added C1: 1uF, Capacitor_SMD:C_0805_2012Metric_Pad1.15x1.40mm_HandSolder, symbol Device:C
- added C2: 0.1uF, Capacitor_SMD:C_0805_2012Metric_Pad1.15x1.40mm_HandSolder, symbol Device:C
- added C4: .1uF, Capacitor_SMD:C_0805_2012Metric_Pad1.15x1.40mm_HandSolder, symbol Device:C
- added D1, D10, D11, D12, D13, D14, D15, D16, D7, D8, D9: LED, Diode_SMD:D_0805_2012Metric_Pad1.15x1.40mm_HandSolder, symbol Device:LED
- added R1: 20k, Resistor_SMD:R_0805_2012Metric_Pad1.15x1.40mm_HandSolder, symbol Device:R
- added U1: IS31FL3731-SA, Package_SO:SSOP-28_5.3x10.2mm_P0.65mm, symbol Driver_LED:IS31FL3731-SA
- D2, D3, D4, D5, D6: footprint LED_SMD:LED_0805_2012Metric -> Diode_SMD:D_0805_2012Metric_Pad1.15x1.40mm_HandSolder
- renumbered C1 to C3, D1 to D17, J6 to J2, R1 to R2, U1 to U2
Connections:
- net +3V3: now also C1.2, C4.2, U1.2 (VCC)
- net GND: now also C1.1, C2.2, C4.1, R1.1, U1.5 (GND); no longer D2.1 (K), D3.1 (K), D4.1 (K), D5.1 (K), D6.1 (K)
- net MOSI: now also U1.19 (SDA)
- net SCK: now also U1.20 (SCL)
- net at D4.2 (A): now also D12.2 (A)
- net at D5.2 (A): now also D13.2 (A)
- net at D3.2 (A): now also D11.2 (A)
- net at D2.2 (A): now also D10.2 (A)
- net at D6.2 (A): now also D14.2 (A)
- new net: C2.1, U1.16 (C_FILT)
- new net: R1.2, U1.6 (R_EXT)
- new net: D16.2 (A), D8.2 (A)
- new net: D15.2 (A), D7.2 (A)
- new net CA1: D1.1 (K), D2.1 (K), D3.1 (K), D4.1 (K), D5.1 (K), D6.1 (K), D7.1 (K), D8.1 (K), D9.2 (A), U1.21 (CA1)
- new net CA2: D1.2 (A), D10.1 (K), D11.1 (K), D12.1 (K), D13.1 (K), D14.1 (K), D15.1 (K), D16.1 (K), D9.1 (K), U1.22 (CA2)
- no-connect marks 0 -> 20
